Commit message: Change joint types from continuous to revolute and add actuator cfg

File: urdf/robit-adult-humanoid.xacro (robot description, xacro)
@@ -284,81 +284,159 @@
   </collision>
 </link>
-<joint name="torso_yaw" type="continuous">
+<!-- ROBSTRIDE06 -->
+<joint name="torso_yaw" type="revolute">
   <origin xyz="-0.012811 -0.00231 0.061621" rpy="0 0 0"/>
   <parent link="base_link"/>
   <child link="torso_dummy_1"/>
   <axis xyz="0.0 -0.0 1.0"/>
-</joint>
-<joint name="left_hip_pitch" type="continuous">
+  <limit
+      lower="0.0"
+      upper="0.0"
+      effort="36"
+      velocity="67.0" />
+</joint>
+<!-- ROBSTRIDE04 -->
+<joint name="left_hip_pitch" type="revolute">
   <origin xyz="-0.012811 0.05519 -0.068879" rpy="0 0 0"/>
   <parent link="base_link"/>
   <child link="left_hip_1"/>
   <axis xyz="0.0 1.0 0.0"/>
-</joint>
-<joint name="left_hip_roll" type="continuous">
+  <limit
+      lower="0"
+      upper="2.34"
+      effort="120.0"
+      velocity="15.0" />
+</joint>
+<!-- ROBSTRIDE03 -->
+<joint name="left_hip_roll" type="revolute">
   <origin xyz="0.03525 0.08 0.0" rpy="0 0 0"/>
   <parent link="left_hip_1"/>
   <child link="left_hip_thigh_1"/>
   <axis xyz="1.0 0.0 0.0"/>
-</joint>
-<joint name="left_knee_pitch" type="continuous">
+  <limit
+      lower="0"
+      upper="2.34"
+      effort="60"
+      velocity="50" />
+</joint>
+<!-- ROBSTRIDE04 -->
+<joint name="left_knee_pitch" type="revolute">
   <origin xyz="-0.02 0.032 -0.1875" rpy="0 0 0"/>
   <parent link="left_thigh_1"/>
   <child link="left_shin_1"/>
   <axis xyz="0.0 1.0 0.0"/>
-</joint>
-<joint name="right_hip_pitch" type="continuous">
+  <limit
+      lower="0"
+      upper="2.34"
+      effort="120.0"
+      velocity="15.0" />
+</joint>
+<!-- ROBSTRIDE04 -->
+<joint name="right_hip_pitch" type="revolute">
   <origin xyz="-0.012811 -0.05981 -0.068879" rpy="0 0 0"/>
   <parent link="base_link"/>
   <child link="right_hip_1"/>
   <axis xyz="0.0 -1.0 -0.0"/>
-</joint>
-<joint name="right_hip_roll" type="continuous">
+  <limit
+      lower="0"
+      upper="2.34"
+      effort="120.0"
+      velocity="15.0" />
+</joint>
+<!-- ROBSTRIDE03 -->
+<joint name="right_hip_roll" type="revolute">
   <origin xyz="0.03525 -0.08 0.0" rpy="0 0 0"/>
   <parent link="right_hip_1"/>
   <child link="right_hip_thigh_1"/>
   <axis xyz="1.0 -0.0 -0.0"/>
-</joint>
-<joint name="left_hip_yaw" type="continuous">
+  <limit
+      lower="0"
+      upper="2.34"
+      effort="60"
+      velocity="50" />
+</joint>
+<!-- ROBSTRIDE03 -->
+<joint name="left_hip_yaw" type="revolute">
   <origin xyz="-0.03425 0.0 -0.11" rpy="0 0 0"/>
   <parent link="left_hip_thigh_1"/>
   <child link="left_thigh_1"/>
   <axis xyz="0.0 0.0 -1.0"/>
-</joint>
-<joint name="right_hip_yaw" type="continuous">
+  <limit
+      lower="0"
+      upper="2.34"
+      effort="60"
+      velocity="50" />
+</joint>
+<!-- ROBSTRIDE03 -->
+<joint name="right_hip_yaw" type="revolute">
   <origin xyz="-0.03425 0.0 -0.11" rpy="0 0 0"/>
   <parent link="right_hip_thigh_1"/>
   <child link="right_thigh_1"/>
   <axis xyz="-0.0 -0.0 -1.0"/>
-</joint>
-<joint name="right_knee_pitch" type="continuous">
+  <limit
+      lower="0"
+      upper="2.34"
+      effort="60"
+      velocity="50" />
+</joint>
+<!-- ROBSTRIDE04 -->
+<joint name="right_knee_pitch" type="revolute">
   <origin xyz="-0.02 -0.032 -0.1875" rpy="0 0 0"/>
   <parent link="right_thigh_1"/>
   <child link="right_shin_1"/>
   <axis xyz="-0.0 -1.0 0.0"/>
-</joint>
-<joint name="left_ankle_pitch" type="continuous">
+  <limit
+      lower="0"
+      upper="2.34"
+      effort="120.0"
+      velocity="15.0" />
+</joint>
+<!-- ROBSTRIDE06 PARREL LINK PIVOT -->
+<joint name="left_ankle_pitch" type="revolute">
   <origin xyz="0.017516 -0.009377 -0.300155" rpy="0 0 0"/>
   <parent link="left_shin_1"/>
   <child link="left_ankle_1"/>
   <axis xyz="-0.0 1.0 0.0"/>
-</joint>
-<joint name="right_ankle_pitch" type="continuous">
+  <limit
+      lower="0"
+      upper="2.34"
+      effort="36"
+      velocity="67.0" />
+</joint>
+<!-- ROBSTRIDE06 PARREL LINK PIVOT -->
+<joint name="right_ankle_pitch" type="revolute">
   <origin xyz="0.017516 0.009377 -0.300155" rpy="0 0 0"/>
   <parent link="right_shin_1"/>
   <child link="right_ankle_1"/>
   <axis xyz="0.0 -1.0 0.0"/>
-</joint>
-<joint name="right_ankle_roll" type="continuous">
+  <limit
+      lower="0"
+      upper="2.34"
+      effort="36"
+      velocity="67.0" />
+</joint>
+<!-- ROBSTRIDE06 PARREL LINK PIVOT -->
+<joint name="right_ankle_roll" type="revolute">
   <origin xyz="0.012 0.0195 0.0" rpy="0 0 0"/>
   <parent link="right_ankle_1"/>
   <child link="right_foot_1"/>
   <axis xyz="1.0 -0.0 0.0"/>
-</joint>
-<joint name="left_ankle_roll" type="continuous">
+  <limit
+      lower="0"
+      upper="2.34"
+      effort="36"
+      velocity="67.0" />
+</joint>
+<!-- ROBSTRIDE06 PARREL LINK PIVOT -->
+<joint name="left_ankle_roll" type="revolute">
   <origin xyz="0.007 -0.0195 0.0" rpy="0 0 0"/>
   <parent link="left_ankle_1"/>
   <child link="left_foot_1"/>
   <axis xyz="1.0 -0.0 0.0"/>
+  <limit
+      lower="0"
+      upper="2.34"
+      effort="36"
+      velocity="67.0" />
 </joint>
 </robot>

Commit message: set link mass

File: urdf/robit-adult-humanoid.xacro (robot description, xacro)
@@ -7,5 +7,5 @@
   <inertial>
     <origin xyz="-0.01281095989310514 -0.0022810841892335573 -0.04582677292819565" rpy="0 0 0"/>
-    <mass value="13.241738959818246"/>
+    <mass value="4.686"/>
     <inertia ixx="0.05322" iyy="0.046518" izz="0.033952" ixy="0.0" iyz="-3.4e-05" ixz="0.0"/>
   </inertial>
@@ -27,5 +27,5 @@
   <inertial>
     <origin xyz="4.010597370179836e-08 2.07269816436019e-08 0.20991445985992171" rpy="0 0 0"/>
-    <mass value="162.68508194775083"/>
+    <mass value="13.0"/>
     <inertia ixx="4.348138" iyy="2.401024" izz="2.407002" ixy="-0.0" iyz="-0.0" ixz="-0.0"/>
   </inertial>
@@ -47,5 +47,5 @@
   <inertial>
     <origin xyz="0.0006297032466040884 0.06724050201455194 -0.00012501074286021263" rpy="0 0 0"/>
-    <mass value="4.7954352907466955"/>
+    <mass value="1.622"/>
     <inertia ixx="0.009165" iyy="0.00579" izz="0.007928" ixy="-3.4e-05" iyz="-1.3e-05" ixz="7e-06"/>
   </inertial>
@@ -67,5 +67,5 @@
   <inertial>
     <origin xyz="-0.03294977172684366 2.0727097427286623e-08 -0.05754189872842047" rpy="0 0 0"/>
-    <mass value="1.2540419749856078"/>
+    <mass value="0.431"/>
     <inertia ixx="0.00238" iyy="0.004152" izz="0.002362" ixy="-0.0" iyz="0.0" ixz="-9.4e-05"/>
   </inertial>
@@ -87,5 +87,5 @@
   <inertial>
     <origin xyz="0.010618528090019137 -0.0333920984187136 -0.14926516145705215" rpy="0 0 0"/>
-    <mass value="5.787046721940419"/>
+    <mass value="2.017"/>
     <inertia ixx="0.03492" iyy="0.034511" izz="0.005734" ixy="-6.6e-05" iyz="-0.00021" ixz="-0.000323"/>
   </inertial>
@@ -107,5 +107,5 @@
   <inertial>
     <origin xyz="0.0006297032483585027 -0.0672404879580738 -0.0001250108063819838" rpy="0 0 0"/>
-    <mass value="4.795435290722294"/>
+    <mass value="1.622"/>
     <inertia ixx="0.009165" iyy="0.00579" izz="0.007928" ixy="3.4e-05" iyz="1.3e-05" ixz="7e-06"/>
   </inertial>
@@ -127,5 +127,5 @@
   <inertial>
     <origin xyz="-0.032949771725187454 2.0726992372432917e-08 -0.0575418987136713" rpy="0 0 0"/>
-    <mass value="1.2540419749867722"/>
+    <mass value="0.431"/>
     <inertia ixx="0.00238" iyy="0.004152" izz="0.002362" ixy="0.0" iyz="-0.0" ixz="-9.4e-05"/>
   </inertial>
@@ -147,5 +147,5 @@
   <inertial>
     <origin xyz="-0.01047227388465445 0.0010136953040755792 -0.12292464330555514" rpy="0 0 0"/>
-    <mass value="10.074283584151052"/>
+    <mass value="3.408"/>
     <inertia ixx="0.066064" iyy="0.069816" izz="0.014807" ixy="9e-05" iyz="0.000661" ixz="-0.006958"/>
   </inertial>
@@ -167,5 +167,5 @@
   <inertial>
     <origin xyz="-0.010472273856055954 -0.0010136538122056948 -0.12292464329228153" rpy="0 0 0"/>
-    <mass value="10.074283584900902"/>
+    <mass value="3.408"/>
     <inertia ixx="0.066064" iyy="0.069816" izz="0.014807" ixy="-9e-05" iyz="-0.000661" ixz="-0.006958"/>
   </inertial>
@@ -187,5 +187,5 @@
   <inertial>
     <origin xyz="0.010618528091643188 0.033392135688315616 -0.1492651614422552" rpy="0 0 0"/>
-    <mass value="5.78704672194055"/>
+    <mass value="2.017"/>
     <inertia ixx="0.03492" iyy="0.034511" izz="0.005734" ixy="6.6e-05" iyz="0.00021" ixz="-0.000323"/>
   </inertial>
@@ -207,5 +207,5 @@
   <inertial>
     <origin xyz="3.640125762864599e-07 -0.019499640616245678 -3.179999508162723e-07" rpy="0 0 0"/>
-    <mass value="0.06598347385516057"/>
+    <mass value="0.036"/>
     <inertia ixx="1.1e-05" iyy="6e-06" izz="1e-05" ixy="-0.0" iyz="-0.0" ixz="-0.0"/>
   </inertial>
@@ -227,5 +227,5 @@
   <inertial>
     <origin xyz="3.640142449499312e-07 0.019499682070422297 -3.179851766343944e-07" rpy="0 0 0"/>
-    <mass value="0.0659834738551606"/>
+    <mass value="0.036"/>
     <inertia ixx="1.1e-05" iyy="6e-06" izz="1e-05" ixy="0.0" iyz="0.0" ixz="0.0"/>
   </inertial>
@@ -247,5 +247,5 @@
   <inertial>
     <origin xyz="0.0002537656221860748 -3.1792990121126685e-07 -0.046881970453633515" rpy="0 0 0"/>
-    <mass value="1.9765556077954949"/>
+    <mass value="0.494"/>
     <inertia ixx="0.001684" iyy="0.003666" izz="0.005031" ixy="0.0" iyz="0.0" ixz="5.8e-05"/>
   </inertial>
@@ -267,5 +267,5 @@
   <inertial>
     <origin xyz="0.005253765620523281 3.5938407663693717e-07 -0.046881970468406475" rpy="0 0 0"/>
-    <mass value="1.9765556077954982"/>
+    <mass value="0.494"/>
     <inertia ixx="0.001684" iyy="0.003666" izz="0.005031" ixy="-0.0" iyz="-0.0" ixz="5.8e-05"/>
   </inertial>
